File: Codex_KiCad_USB_UART_Demo/hardware/USB_UART_Bridge/Power.kicad_sch (KiCad schematic)
At the start: 10 parts, among them U4 AP2112K-3.3

Commit message: feat: complete USB UART PCB layout and routing
Parts:
- PS1: value CRE1S0505SC -> IB0505LS-1WR3; footprint Converter_DCDC:Converter_DCDC_Murata_CRE1xxxxxxSC_THT -> USB_UART_Bridge:Converter_DCDC_YLPTEC_IB0505LS-1WR3; symbol Converter_DCDC_Isolated:CRE1S0505SC -> USB_UART_Bridge:IB0505LS-1WR3
Other:
- note added: "PS1: IB0505LS-1WR3 / isolated 1W C7: PS1 +VIN input decoupling 10uF C8: PS1 +VOUT output decoupling 10uF"
- note added: "U4: AP2112K-3.3 / SOT-23-5 / 3.3V / 600mA C9: U4 VOUT 100nF bypass, place at pin5/GND C10: U4 VOUT 10uF filter/bulk, place at pin5/GND"
- note removed: "PS1: CRE1S0505SC / 1W / 1.5kVrms / isolated"
- note removed: "U4: AP2112K-3.3 / SOT-23-5 / 3.3V / 600mA"
Changed lines of the file:
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@@
 	(title_block
 		(title "Power")
+		(date "2026-09-19")
 		(rev "0.2")
-		(date "2026-09-19")
-	)
-	(text "U4: AP2112K-3.3 / SOT-23-5 / 3.3V / 600mA"
+	)
+	(text "U4: AP2112K-3.3 / SOT-23-5 / 3.3V / 600mA\nC9: U4 VOUT 100nF bypass, place at pin5/GND\nC10: U4 VOUT 10uF filter/bulk, place at pin5/GND"
 		(exclude_from_sim no)
 		(at 227.33 111.252 0)
@@
 		)
 	)
-	(text "PS1: CRE1S0505SC / 1W / 1.5kVrms / isolated"
+	(text "PS1: IB0505LS-1WR3 / isolated 1W\nC7: PS1 +VIN input decoupling 10uF\nC8: PS1 +VOUT output decoupling 10uF"
 		(exclude_from_sim no)
 		(at 135.128 114.046 0)
@@
 		(pts
 			(xy 48.26 93.98) (xy 62.23 93.98)
+		)
+		(stroke
+			(width 0)
+			(type default)
+		)
+	)
+	(wire
+		(pts
+			(xy 62.23 88.9) (xy 62.23 83.82)
 		)
 		(stroke
@@
 			)
 			(project "USB_UART_Bridge"
-				(path "/6d719abe-8294-4a13-afeb-1c2f95178f03/734a3fd4-b022-4fbc-bb04-e2dac4c1f1f0"
+				(path "/991ad087-5b84-4353-b5af-12ada82ec90c/734a3fd4-b022-4fbc-bb04-e2dac4c1f1f0"
 					(reference "C1")
 					(unit 1)
@@
 			)
 			(project "USB_UART_Bridge"
-				(path "/6d719abe-8294-4a13-afeb-1c2f95178f03/734a3fd4-b022-4fbc-bb04-e2dac4c1f1f0"
+				(path "/991ad087-5b84-4353-b5af-12ada82ec90c/734a3fd4-b022-4fbc-bb04-e2dac4c1f1f0"
 					(reference "#PWR006")
 					(unit 1)
@@
 			)
 			(project "USB_UART_Bridge"
-				(path "/6d719abe-8294-4a13-afeb-1c2f95178f03/734a3fd4-b022-4fbc-bb04-e2dac4c1f1f0"
+				(path "/991ad087-5b84-4353-b5af-12ada82ec90c/734a3fd4-b022-4fbc-bb04-e2dac4c1f1f0"
 					(reference "C10")
 					(unit 1)
@@
 			)
 			(project "USB_UART_Bridge"
-				(path "/6d719abe-8294-4a13-afeb-1c2f95178f03/734a3fd4-b022-4fbc-bb04-e2dac4c1f1f0"
+				(path "/991ad087-5b84-4353-b5af-12ada82ec90c/734a3fd4-b022-4fbc-bb04-e2dac4c1f1f0"
 					(reference "U4")
 					(unit 1)
@@
 			)
 			(project "USB_UART_Bridge"
-				(path "/6d719abe-8294-4a13-afeb-1c2f95178f03/734a3fd4-b022-4fbc-bb04-e2dac4c1f1f0"
+				(path "/991ad087-5b84-4353-b5af-12ada82ec90c/734a3fd4-b022-4fbc-bb04-e2dac4c1f1f0"
 					(reference "TP1")
 					(unit 1)
@@
 			)
 			(project "USB_UART_Bridge"
-				(path "/6d719abe-8294-4a13-afeb-1c2f95178f03/734a3fd4-b022-4fbc-bb04-e2dac4c1f1f0"
+				(path "/991ad087-5b84-4353-b5af-12ada82ec90c/734a3fd4-b022-4fbc-bb04-e2dac4c1f1f0"
 					(reference "#PWR003")
 					(unit 1)
@@
 			)
 			(project "USB_UART_Bridge"
-				(path "/6d719abe-8294-4a13-afeb-1c2f95178f03/734a3fd4-b022-4fbc-bb04-e2dac4c1f1f0"
+				(path "/991ad087-5b84-4353-b5af-12ada82ec90c/734a3fd4-b022-4fbc-bb04-e2dac4c1f1f0"
 					(reference "#PWR009")
 					(unit 1)
@@
 			)
 			(project "USB_UART_Bridge"
-				(path "/6d719abe-8294-4a13-afeb-1c2f95178f03/734a3fd4-b022-4fbc-bb04-e2dac4c1f1f0"
+				(path "/991ad087-5b84-4353-b5af-12ada82ec90c/734a3fd4-b022-4fbc-bb04-e2dac4c1f1f0"
 					(reference "TP2")
 					(unit 1)
@@
 			)
 			(project "USB_UART_Bridge"
-				(path "/6d719abe-8294-4a13-afeb-1c2f95178f03/734a3fd4-b022-4fbc-bb04-e2dac4c1f1f0"
+				(path "/991ad087-5b84-4353-b5af-12ada82ec90c/734a3fd4-b022-4fbc-bb04-e2dac4c1f1f0"
 					(reference "#PWR012")
 					(unit 1)
@@
 			)
 			(project "USB_UART_Bridge"
-				(path "/6d719abe-8294-4a13-afeb-1c2f95178f03/734a3fd4-b022-4fbc-bb04-e2dac4c1f1f0"
+				(path "/991ad087-5b84-4353-b5af-12ada82ec90c/734a3fd4-b022-4fbc-bb04-e2dac4c1f1f0"
 					(reference "#PWR011")
 					(unit 1)
@@
 			)
 			(project "USB_UART_Bridge"
-				(path "/6d719abe-8294-4a13-afeb-1c2f95178f03/734a3fd4-b022-4fbc-bb04-e2dac4c1f1f0"
+				(path "/991ad087-5b84-4353-b5af-12ada82ec90c/734a3fd4-b022-4fbc-bb04-e2dac4c1f1f0"
 					(reference "#PWR008")
+					(unit 1)
+				)
+			)
+		)
+	)
+	(symbol
+		(lib_id "power:PWR_FLAG")
+		(at 62.23 83.82 0)
+		(unit 1)
+		(body_style 1)
+		(exclude_from_sim no)
+		(in_bom yes)
+		(on_board yes)
+		(in_pos_files yes)
+		(dnp no)
+		(property "Reference" "#FLG005"
+			(at 62.23 85.725 0)
+			(hide yes)
+			(show_name no)
+			(do_not_autoplace no)
+			(effects
+				(font
+					(size 1.27 1.27)
+				)
+				(justify left)
+			)
+		)
+		(property "Value" "PWR_FLAG"
+			(at 62.23 78.74 0)
+			(show_name no)
+			(do_not_autoplace no)
+			(effects
+				(font
+					(size 1.27 1.27)
+				)
+			)
+		)
+		(property "Footprint" ""
+			(at 62.23 83.82 0)
+			(show_name no)
+			(do_not_autoplace no)
+			(effects
+				(font
+					(size 1.27 1.27)
+				)
+			)
+		)
+		(property "Datasheet" ""
+			(at 62.23 83.82 0)
+			(show_name no)
+			(do_not_autoplace no)
+			(effects
+				(font
+					(size 1.27 1.27)
+				)
+			)
+		)
+		(property "Description" ""
+			(at 62.23 83.82 0)
+			(show_name no)
+			(do_not_autoplace no)
+			(effects
+				(font
+					(size 1.27 1.27)
+				)
+			)
+		)
+		(pin "1"
+		)
+		(instances
+			(project ""
+				(path "/635ef601-7197-43f9-8c20-a7525b81003e"
+					(reference "#FLG005")
+					(unit 1)
+				)
+			)
+			(project "USB_UART_Bridge"
+				(path "/991ad087-5b84-4353-b5af-12ada82ec90c/734a3fd4-b022-4fbc-bb04-e2dac4c1f1f0"
+					(reference "#FLG005")
 					(unit 1)
 				)
@@
 			)
 			(project "USB_UART_Bridge"
-				(path "/6d719abe-8294-4a13-afeb-1c2f95178f03/734a3fd4-b022-4fbc-bb04-e2dac4c1f1f0"
+				(path "/991ad087-5b84-4353-b5af-12ada82ec90c/734a3fd4-b022-4fbc-bb04-e2dac4c1f1f0"
 					(reference "#PWR017")
 					(unit 1)
@@
 			)
 			(project "USB_UART_Bridge"
-				(path "/6d719abe-8294-4a13-afeb-1c2f95178f03/734a3fd4-b022-4fbc-bb04-e2dac4c1f1f0"
+				(path "/991ad087-5b84-4353-b5af-12ada82ec90c/734a3fd4-b022-4fbc-bb04-e2dac4c1f1f0"
 					(reference "C8")
 					(unit 1)
@@
 			)
 			(project "USB_UART_Bridge"
-				(path "/6d719abe-8294-4a13-afeb-1c2f95178f03/734a3fd4-b022-4fbc-bb04-e2dac4c1f1f0"
+				(path "/991ad087-5b84-4353-b5af-12ada82ec90c/734a3fd4-b022-4fbc-bb04-e2dac4c1f1f0"
 					(reference "#PWR014")
 					(unit 1)
@@
 			)
 			(project "USB_UART_Bridge"
-				(path "/6d719abe-8294-4a13-afeb-1c2f95178f03/734a3fd4-b022-4fbc-bb04-e2dac4c1f1f0"
+				(path "/991ad087-5b84-4353-b5af-12ada82ec90c/734a3fd4-b022-4fbc-bb04-e2dac4c1f1f0"
 					(reference "C7")
 					(unit 1)
@@
 			)
 			(project "USB_UART_Bridge"
-				(path "/6d719abe-8294-4a13-afeb-1c2f95178f03/734a3fd4-b022-4fbc-bb04-e2dac4c1f1f0"
+				(path "/991ad087-5b84-4353-b5af-12ada82ec90c/734a3fd4-b022-4fbc-bb04-e2dac4c1f1f0"
 					(reference "F1")
 					(unit 1)
@@
 			)
 			(project "USB_UART_Bridge"
-				(path "/6d719abe-8294-4a13-afeb-1c2f95178f03/734a3fd4-b022-4fbc-bb04-e2dac4c1f1f0"
+				(path "/991ad087-5b84-4353-b5af-12ada82ec90c/734a3fd4-b022-4fbc-bb04-e2dac4c1f1f0"
 					(reference "#PWR016")
 					(unit 1)
@@
 			)
 			(project "USB_UART_Bridge"
-				(path "/6d719abe-8294-4a13-afeb-1c2f95178f03/734a3fd4-b022-4fbc-bb04-e2dac4c1f1f0"
+				(path "/991ad087-5b84-4353-b5af-12ada82ec90c/734a3fd4-b022-4fbc-bb04-e2dac4c1f1f0"
 					(reference "#PWR004")
 					(unit 1)
@@
 			)
 			(project "USB_UART_Bridge"
-				(path "/6d719abe-8294-4a13-afeb-1c2f95178f03/734a3fd4-b022-4fbc-bb04-e2dac4c1f1f0"
+				(path "/991ad087-5b84-4353-b5af-12ada82ec90c/734a3fd4-b022-4fbc-bb04-e2dac4c1f1f0"
 					(reference "C9")
 					(unit 1)
@@
 			)
 			(project "USB_UART_Bridge"
-				(path "/6d719abe-8294-4a13-afeb-1c2f95178f03/734a3fd4-b022-4fbc-bb04-e2dac4c1f1f0"
+				(path "/991ad087-5b84-4353-b5af-12ada82ec90c/734a3fd4-b022-4fbc-bb04-e2dac4c1f1f0"
 					(reference "#PWR001")
 					(unit 1)
@@
 	)
 	(symbol
-		(lib_id "Converter_DCDC_Isolated:CRE1S0505SC")
+		(lib_id "USB_UART_Bridge:IB0505LS-1WR3")
 		(at 132.08 101.6 0)
 		(unit 1)
@@
 			)
 		)
-		(property "Value" "CRE1S0505SC"
+		(property "Value" "IB0505LS-1WR3"
 			(at 134.62 110.49 0)
 			(show_name no)
@@
 			)
 		)
-		(property "Footprint" "Converter_DCDC:Converter_DCDC_Murata_CRE1xxxxxxSC_THT"
+		(property "Footprint" "USB_UART_Bridge:Converter_DCDC_YLPTEC_IB0505LS-1WR3"
 			(at 132.08 91.44 0)
 			(hide yes)
@@
 			)
 		)
-		(property "Datasheet" ""
+		(property "Datasheet" "https://item.szlcsc.com/6212649.html"
 			(at 132.08 101.6 0)
 			(show_name no)
@@
 			)
 		)
-		(property "Description" ""
-			(at 132.08 101.6 0)
+		(property "Description" "5V to 5V 200mA isolated DC-DC converter, 1W, SIP-4"
+			(at 133.35 119.126 0)
 			(show_name no)
 			(do_not_autoplace no)
@@
 			)
 			(project "USB_UART_Bridge"
-				(path "/6d719abe-8294-4a13-afeb-1c2f95178f03/734a3fd4-b022-4fbc-bb04-e2dac4c1f1f0"
+				(path "/991ad087-5b84-4353-b5af-12ada82ec90c/734a3fd4-b022-4fbc-bb04-e2dac4c1f1f0"
 					(reference "PS1")
 					(unit 1)
@@
 			)
 			(project "USB_UART_Bridge"
-				(path "/6d719abe-8294-4a13-afeb-1c2f95178f03/734a3fd4-b022-4fbc-bb04-e2dac4c1f1f0"
+				(path "/991ad087-5b84-4353-b5af-12ada82ec90c/734a3fd4-b022-4fbc-bb04-e2dac4c1f1f0"
 					(reference "#PWR013")
 					(unit 1)
