File: LA150C_DRIVER_V1.00/硬件相关/Project/LA150C_RDIVER_V1.00/SCH_LA150C_ENCODER_V1.00.kicad_sch (KiCad schematic)
At the start: 3 parts, among them U2 MT6701

Commit message: chore: save LA150C schematic updates
Parts:
- renumbered C11 to C31, C12 to C32, U2 to U4
Other:
- moved on the sheet: C31, C32, U4
